File: Section A - Title A.kicad_sch (KiCad schematic)
At the start: 4 parts

Commit message: section-a: R304 + fragment
Parts:
- added R304: 68k, Resistor_SMD:R_0603_1608Metric, symbol Device:R
Changed lines of the file:
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@@
+		)
+	)
+	(symbol
+		(lib_id "Device:R")
+		(at 152.4 101.6 0)
+		(unit 1)
+		(exclude_from_sim no)
+		(in_bom yes)
+		(on_board yes)
+		(dnp no)
+		(property "Reference" "R304"
+			(at 154.94 101.6 0)
+			(effects (font (size 1.27 1.27)) (justify left))
+		)
+		(property "Value" "68k"
+			(at 154.94 104.14 0)
+			(effects (font (size 1.27 1.27)) (justify left))
+		)
+		(property "Footprint" "Resistor_SMD:R_0603_1608Metric"
+			(at 152.4 101.6 0)
+			(effects (font (size 1.27 1.27)) (hide yes))
+		)
+		(property "Datasheet" "~"
+			(at 152.4 101.6 0)
+			(effects (font (size 1.27 1.27)) (hide yes))
+		)
+		(pin "1")
+		(pin "2")
+		(instances
+			(project "ci_dummy"
+				(path "/f9e05184-c88b-4a88-ae9c-ab2bdb32be7c/c5103ceb-5325-4a84-a025-9638a412984e/f06537ee-772d-44d3-8c50-e0ba41038c9c"
+					(reference "R304")
+					(unit 1)
+				)
+			)
 		)
 	)

Commit message: dev: no-connects + footprints for R304/R405 before release
Connections:
- no-connect marks 8 -> 10
Changed lines of the file:
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@@
 		(at 132.08 105.41)
+	)
+	(no_connect
+		(at 152.4 97.79)
+	)
+	(no_connect
+		(at 152.4 105.41)
 	)
 	(symbol
